Commit message: Respawn boxes

File: urdf/kinova_g3l_box_picker.urdf.xacro (robot description, xacro)
@@ -25,10 +25,8 @@
   <xacro:arg name="sim_isaac" default="false" />
   <xacro:arg name="gazebo_renderer" default="ogre"/>
-  <xacro:arg name="camera_width" default="640"/>
-  <xacro:arg name="camera_height" default="480"/>
-  <xacro:arg name="camera_fps" default="6"/>
   <xacro:arg name="simulation_controllers" default="$(find easy_kinova_g3l_moveit_config)/config/ros2_controllers.yaml" />
   <xacro:arg name="moveit_active" default="false"/>
   <!-- import main macro -->
+  <xacro:include filename="$(find easy_simulation)/urdf/rgbd_camera.urdf.xacro" />
   <xacro:include filename="$(find kortex_description)/robots/kortex_robot.xacro" />
   <!-- initial position for simulations (Mock Hardware, Gazebo) -->
@@ -77,66 +75,15 @@
       </plugin>
     </gazebo>
-    <gazebo reference="camera_color_frame">
-      <sensor name="camera_sensor" type="rgbd_camera">
-        <camera>
-          <horizontal_fov>1.047</horizontal_fov>
-          <image>
-            <width>$(arg camera_width)</width>
-            <height>$(arg camera_height)</height>
-            <format>RGB_INT8</format>
-          </image>
-          <clip>
-            <near>0.1</near>
-            <far>5</far>
-          </clip>
-          <distortion>
-            <k1>0.0</k1>
-            <k2>0.0</k2>
-            <k3>0.0</k3>
-            <p1>0.0</p1>
-            <p2>0.0</p2>
-            <center>0.5 0.5</center>
-          </distortion>
-          <lens>
-            <intrinsics>
-              <fx>554.25469</fx>
-              <fy>554.25469</fy>
-              <cx>320.5</cx>
-              <cy>240.5</cy>
-              <s>0</s>
-            </intrinsics>
-            <!-- These need to match the intrinsics above or
-            Gazebo will default to different default values -->
-            <projection>
-              <p_fx>554.25469</p_fx>
-              <p_fy>554.25469</p_fy>
-              <p_cx>320.5</p_cx>
-              <p_cy>240.5</p_cy>
-              <tx>0</tx>
-              <ty>0</ty>
-            </projection>
-          </lens>
-          <noise>
-            <type>gaussian</type>
-            <mean>0</mean>
-            <stddev>0.00</stddev>
-          </noise>
-          <depth_camera>
-            <clip>
-              <near>0.25</near>
-              <far>5</far>
-            </clip>
-          </depth_camera>
-          <optical_frame_id>color_optical_frame</optical_frame_id>
-        </camera>
-        <gz_frame_id>camera_color_frame</gz_frame_id>
-        <always_on>1</always_on>
-        <update_rate>$(arg camera_fps)</update_rate>
-        <visualize>true</visualize>
-        <topic>wrist_mounted_camera</topic>
-        <enable_metrics>false</enable_metrics>
-      </sensor>
-    </gazebo>
+    <xacro:gz_rgbd_camera
+      name="camera"
+      prefix="$(arg prefix)"/>
   </xacro:if>
+  <!-- RGBD camera URDF inclusion -->
+  <xacro:rgbd_camera
+    parent_link="$(arg prefix)base_link"
+    name="camera"
+    prefix="$(arg prefix)">
+    <origin xyz="0.2 0 1.2" rpy="0 1.2 0"/>
+  </xacro:rgbd_camera>
   <!-- Suction gripper URDF inclusion -->
   <link name="$(arg prefix)suction_gripper_base">

File: worlds/box_picking_desk.sdf.xacro (robot description, xacro)
@@ -1,3 +1,5 @@
-<sdf version='1.10'>
+<?xml version="1.0"?>
+<sdf version='1.10'
+    xmlns:xacro="http://ros.org/wiki/xacro">
   <world name='empty'>
     <physics name='1ms' type='ignored'>
@@ -10,4 +12,5 @@
     <plugin name='gz::sim::systems::SceneBroadcaster' filename='gz-sim-scene-broadcaster-system'/>
     <plugin name='gz::sim::systems::Contact' filename='gz-sim-contact-system'/>
+    <plugin filename="libros_gz_sim.so" name="ros_gz_sim"/>
     <gravity>0 0 -9.8000000000000007</gravity>
     <magnetic_field>5.5644999999999998e-06 2.2875799999999999e-05 -4.2388400000000002e-05</magnetic_field>
@@ -251,5 +254,5 @@
         <enable_wind>false</enable_wind>
       </link>
-      <pose>0 0 0 0 0 1.57079</pose>
+      <pose>0 0 0 0 0 1.5707900000000004</pose>
       <self_collide>false</self_collide>
     </model>
@@ -438,7 +441,23 @@
         <enable_wind>false</enable_wind>
       </link>
-      <pose>0.8 0.0 0 0 0 1.57079</pose>
+      <pose>0.80000000000000004 0 0 0 0 1.5707900000000004</pose>
       <self_collide>false</self_collide>
     </model>
+    <xacro:macro name="box" params="name origin">
+      <include>
+        <uri>file:///$(find easy_simulation)/worlds/models/cardboard_box</uri>
+        <name>${name}</name>
+        <pose>${origin}</pose>
+      </include>
+    </xacro:macro>
+    <xacro:macro name="target_box" params="name origin">
+      <include>
+        <uri>file:///$(find easy_simulation)/worlds/models/cardboard_box_green</uri>
+        <name>${name}</name>
+        <pose>${origin}</pose>
+      </include>
+    </xacro:macro>
+    <xacro:box name="box1" origin="0.87095397710800171 -0.021143499761819839 1.1649983722855026 0 0 0" />
+    <xacro:target_box name="target_box1" origin="0.87095397710800171 -0.5 1.1649983722855026 0 0 0" />
     <light name='sun' type='directional'>
       <pose>0 0 10 0 0 0</pose>

Commit message: Done vacuum gripper

File: urdf/kinova_g3l_box_picker.urdf.xacro (robot description, xacro)
@@ -24,5 +24,5 @@
   <xacro:arg name="sim_gazebo" default="true" />
   <xacro:arg name="sim_isaac" default="false" />
-  <xacro:arg name="gazebo_renderer" default="ogre"/>
+  <xacro:arg name="gazebo_renderer" default="ogre2"/>
   <xacro:arg name="simulation_controllers" default="$(find easy_kinova_g3l_moveit_config)/config/ros2_controllers.yaml" />
   <xacro:arg name="moveit_active" default="false"/>
@@ -87,39 +87,5 @@
   </xacro:rgbd_camera>
   <!-- Suction gripper URDF inclusion -->
-  <link name="$(arg prefix)suction_gripper_base">
-    <inertial>
-      <mass value="0.2" />
-      <origin xyz="0 0 0" rpy="0 0 0" />
-      <inertia
-        ixx="0.0001" ixy="0.0" ixz="0.0"
-        iyy="0.0001" iyz="0.0"
-        izz="0.0001" />
-    </inertial>
-    <visual>
-      <origin xyz="0 0 0" rpy="0 0 0" />
-      <geometry>
-        <mesh filename="file://$(find easy_simulation)/urdf/suction_gripper.stl" scale="0.5 0.5 0.5" />
-      </geometry>
-      <material name="gray">
-        <color rgba="0.5 0.5 0.5 1.0" />
-      </material>
-    </visual>
-    <collision>
-      <origin xyz="0 0 .05" rpy="0 0 0" />
-      <geometry>
-        <box size="0.12 0.05 0.08" />
-      </geometry>
-    </collision>
-  </link>
-  <joint name="$(arg prefix)suction_gripper_joint" type="fixed">
-    <parent link="$(arg prefix)end_effector_link" />
-    <child link="$(arg prefix)suction_gripper_base" />
-    <origin xyz="0 0 0.03" rpy="0 0 0" />
-  </joint>
-  <link name="virtual_suction_tip" />
-  <joint name="virtual_suction_tip_joint" type="fixed">
-    <parent link="$(arg prefix)suction_gripper_base" />
-    <child link="virtual_suction_tip" />
-    <origin xyz="0 0 0.1" rpy="0 0 0" />
-  </joint>
+  <xacro:include filename="$(find easy_simulation)/urdf/suction_gripper.urdf.xacro" />
+  <xacro:suction_gripper prefix="$(arg prefix)" />
 </robot>

File: urdf/rgbd_camera.urdf.xacro (robot description, xacro)
@@ -7,9 +7,19 @@
         <!-- Camera link -->
         <link name="${prefix}${name}_frame">
-            <!-- <visual>
+            <visual>
                 <geometry>
-                    <box size="0.05 0.05 0.05" />
+                    <mesh filename="file://$(find easy_simulation)/urdf/zed2.stl" />
                 </geometry>
-            </visual> -->
+                <material name="dark_gray">
+                    <ambient>0.05 0.05 0.05 1</ambient>
+                    <diffuse>0.05 0.05 0.05 1</diffuse>
+                    <specular>0.01 0.01 0.01 1</specular>
+                    <pbr type="metal">
+                        <albedo>0.05 0.05 0.05 1</albedo>
+                        <metalness>0.2</metalness>
+                        <roughness>0.9</roughness>
+                    </pbr>
+                </material>
+            </visual>
         </link>
         <!-- Fixed joint connecting camera to parent -->

File: worlds/box_picking_desk.sdf.xacro (robot description, xacro)
@@ -1,5 +1,5 @@
 <?xml version="1.0"?>
 <sdf version='1.10'
-    xmlns:xacro="http://ros.org/wiki/xacro">
+  xmlns:xacro="http://ros.org/wiki/xacro">
   <world name='empty'>
     <physics name='1ms' type='ignored'>
@@ -8,12 +8,28 @@
       <real_time_update_rate>1000</real_time_update_rate>
     </physics>
-    <plugin name='gz::sim::systems::Physics' filename='gz-sim-physics-system'/>
-    <plugin name='gz::sim::systems::UserCommands' filename='gz-sim-user-commands-system'/>
-    <plugin name='gz::sim::systems::SceneBroadcaster' filename='gz-sim-scene-broadcaster-system'/>
-    <plugin name='gz::sim::systems::Contact' filename='gz-sim-contact-system'/>
-    <plugin filename="libros_gz_sim.so" name="ros_gz_sim"/>
+    <plugin
+      filename="gz-sim-physics-system"
+      name="gz::sim::systems::Physics">
+    </plugin>
+    <plugin
+      filename="gz-sim-user-commands-system"
+      name="gz::sim::systems::UserCommands">
+    </plugin>
+    <plugin
+      filename="gz-sim-scene-broadcaster-system"
+      name="gz::sim::systems::SceneBroadcaster">
+    </plugin>
+    <plugin
+      filename="gz-sim-imu-system"
+      name="gz::sim::systems::Imu">
+    </plugin>
+    <plugin
+      filename="gz-sim-contact-system"
+      name="gz::sim::systems::Contact">
+    </plugin>
+    <plugin filename="libros_gz_sim.so" name="ros_gz_sim" />
     <gravity>0 0 -9.8000000000000007</gravity>
     <magnetic_field>5.5644999999999998e-06 2.2875799999999999e-05 -4.2388400000000002e-05</magnetic_field>
-    <atmosphere type='adiabatic'/>
+    <atmosphere type='adiabatic' />
     <scene>
       <ambient>0.400000006 0.400000006 0.400000006 1</ambient>
@@ -33,8 +49,8 @@
           <surface>
             <friction>
-              <ode/>
-            </friction>
-            <bounce/>
-            <contact/>
+              <ode />
+            </friction>
+            <bounce />
+            <contact />
           </surface>
         </collision>
@@ -87,6 +103,6 @@
               </ode>
             </friction>
-            <bounce/>
-            <contact/>
+            <bounce />
+            <contact />
           </surface>
         </collision>
@@ -106,5 +122,6 @@
             <pbr>
               <metal>
-                <albedo_map>https://fuel.gazebosim.org/1.0/openrobotics/models/table/4/files/Table_Diffuse.jpg</albedo_map>
+                <albedo_map>
+                  https://fuel.gazebosim.org/1.0/openrobotics/models/table/4/files/Table_Diffuse.jpg</albedo_map>
               </metal>
             </pbr>
@@ -121,8 +138,8 @@
           <surface>
             <friction>
-              <ode/>
-            </friction>
-            <bounce/>
-            <contact/>
+              <ode />
+            </friction>
+            <bounce />
+            <contact />
           </surface>
         </collision>
@@ -153,8 +170,8 @@
           <surface>
             <friction>
-              <ode/>
-            </friction>
-            <bounce/>
-            <contact/>
+              <ode />
+            </friction>
+            <bounce />
+            <contact />
           </surface>
         </collision>
@@ -185,8 +202,8 @@
           <surface>
             <friction>
-              <ode/>
-            </friction>
-            <bounce/>
-            <contact/>
+              <ode />
+            </friction>
+            <bounce />
+            <contact />
           </surface>
         </collision>
@@ -217,8 +234,8 @@
           <surface>
             <friction>
-              <ode/>
-            </friction>
-            <bounce/>
-            <contact/>
+              <ode />
+            </friction>
+            <bounce />
+            <contact />
           </surface>
         </collision>
@@ -274,6 +291,6 @@
               </ode>
             </friction>
-            <bounce/>
-            <contact/>
+            <bounce />
+            <contact />
           </surface>
         </collision>
@@ -293,5 +310,6 @@
             <pbr>
               <metal>
-                <albedo_map>https://fuel.gazebosim.org/1.0/openrobotics/models/table/4/files/Table_Diffuse.jpg</albedo_map>
+                <albedo_map>
+                  https://fuel.gazebosim.org/1.0/openrobotics/models/table/4/files/Table_Diffuse.jpg</albedo_map>
               </metal>
             </pbr>
@@ -308,8 +326,8 @@
           <surface>
             <friction>
-              <ode/>
-            </friction>
-            <bounce/>
-            <contact/>
+              <ode />
+            </friction>
+            <bounce />
+            <contact />
           </surface>
         </collision>
@@ -340,8 +358,8 @@
           <surface>
             <friction>
-              <ode/>
-            </friction>
-            <bounce/>
-            <contact/>
+              <ode />
+            </friction>
+            <bounce />
+            <contact />
           </surface>
         </collision>
@@ -372,8 +390,8 @@
           <surface>
             <friction>
-              <ode/>
-            </friction>
-            <bounce/>
-            <contact/>
+              <ode />
+            </friction>
+            <bounce />
+            <contact />
           </surface>
         </collision>
@@ -404,8 +422,8 @@
           <surface>
             <friction>
-              <ode/>
-            </friction>
-            <bounce/>
-            <contact/>
+              <ode />
+            </friction>
+            <bounce />
+            <contact />
           </surface>
         </collision>
@@ -440,4 +458,9 @@
         </inertial>
         <enable_wind>false</enable_wind>
+        <sensor name='sensor_contact' type='contact'>
+          <contact>
+            <collision>surface</collision>
+          </contact>
+        </sensor>
       </link>
       <pose>0.80000000000000004 0 0 0 0 1.5707900000000004</pose>
@@ -458,6 +481,11 @@
       </include>
     </xacro:macro>
-    <xacro:box name="box1" origin="0.87095397710800171 -0.021143499761819839 1.1649983722855026 0 0 0" />
+    <xacro:box name="box1"
+      origin="0.87095397710800171 -0.021143499761819839 1.1649983722855026 0 0 0" />
     <xacro:target_box name="target_box1" origin="0.87095397710800171 -0.5 1.1649983722855026 0 0 0" />
+    <!-- <plugin
+        filename="easy_simulation_plugins"
+        name="easy_simulation_plugins::SuctionGripperPlugin">
+    </plugin> -->
     <light name='sun' type='directional'>
       <pose>0 0 10 0 0 0</pose>
